File: boards/PoE_Stepper_Driver/PoE_Stepper_Driver.kicad_pcb (KiCad board)
At the start: 2 copper layers, 122 parts, among them J1 RJ45, J2 Motor, J3 Limits, Q1 NMOS_POE, Q10 NMOS_POE, Q3 NMOS_POE, Q4 NMOS_POE, Q5 NMOS_POE, Q6 NMOS_POE, Q7 NMOS_POE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

Commit message: motor control draft 1 done, remember to add capacitor C2 and be mindful of adding connection to power
Parts:
- moved C19 384.9 mm to (35.0, 138.6), turned to 90 degrees
- moved C23 368.6 mm to (44.8, 148.3), turned to 180 degrees
- moved R29 364.2 mm to (49.0, 152.3), turned to 180 degrees
- moved C21 361.4 mm to (58.0, 138.8), turned to 90 degrees
- moved R28 359.8 mm to (53.5, 149.2), turned to 180 degrees
- moved C16 359.2 mm to (54.1, 152.4)
- moved J2 356.8 mm to (43.4, 127.2)
- moved C15 356.8 mm to (44.4, 153.4)
- moved U16 355.0 mm to (46.5, 140.2)
- moved R26 353.8 mm to (38.8, 149.1)
- moved C17 351.2 mm to (46.1, 131.9), turned to 0 degrees
- moved R27 351.1 mm to (39.9, 153.4)
- moved C14 349.1 mm to (53.0, 131.9), turned to 0 degrees
- moved C20 348.6 mm to (65.6, 133.9)
- moved C22 347.8 mm to (65.6, 137.9)
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Routing:
- net GND: track 105.2 -> 24.8 mm, vias 4 -> 16
- net Net-(J3-Pad3): track 0.00 -> 25.0 mm
- net +3V3: track 9.36 -> 32.2 mm
- net Net-(C16-Pad1): track 31.9 -> 11.3 mm
- net Net-(J2-Pad2): track 21.9 -> 41.5 mm, vias 2 -> 0
- net Net-(J2-Pad1): track 38.0 -> 18.6 mm
- net Net-(C23-Pad2): track 21.1 -> 2.28 mm, vias 2 -> 0
- net Net-(J3-Pad4): track 0.00 -> 18.2 mm
- net +12V: track 51.7 -> 66.3 mm, vias 0 -> 11
- net Net-(R28-Pad1): track 35.2 -> 23.6 mm
- net Net-(J2-Pad3): track 29.8 -> 21.7 mm, vias 2 -> 0
- net Net-(C18-Pad2): track 15.1 -> 23.1 mm
- net Net-(J2-Pad4): track 24.6 -> 31.3 mm, vias 2 -> 0
- net Net-(R25-Pad2): track 0.00 -> 6.63 mm
- net Net-(R26-Pad1): track 12.2 -> 16.3 mm, vias 0 -> 2
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- added copper zone on B.Cu, net GND
- added copper zone on F.Cu, net Net-(J2-Pad1)
- added copper zone on F.Cu, net Net-(J2-Pad2)
- added copper zone on F.Cu, net Net-(J2-Pad3)
- added copper zone on F.Cu, net Net-(J2-Pad4)
- removed copper zone on B.Cu, net VOUT-
